Commit message: backup commit not working

File: xacro/wheel_macro.xacro (robot description, xacro)
@@ -60,5 +60,5 @@
 				<plugin>gazebo_ros2_control/GazeboSystem</plugin>
 			</hardware>
-			<joint name="{prefix}_rotate_joint">
+			<joint name="${prefix}_rotate_joint">
 				<command_interface name="position">
 					<param name="min">-15</param>
@@ -71,5 +71,5 @@
 				<state_interface name="effort"/>
 			</joint>
-			<joint name="{prefix}_wheel_joint">
+			<joint name="${prefix}_wheel_joint">
 				<command_interface name="velocity">
 					<param name="min">-20</param>

Commit message: move temporary

File: xacro/wheel_macro.xacro (robot description, xacro)
@@ -56,29 +56,4 @@
 			<kd value="10"/>
 		</gazebo>
-		<!--<ros2_control name="GazeboSystem" type="system">
-			<hardware>
-				<plugin>gazebo_ros2_control/GazeboSystem</plugin>
-			</hardware>
-			<joint name="${prefix}_rotate_joint">
-				<command_interface name="position">
-					<param name="min">-15</param>
-					<param name="max">15</param>
-				</command_interface>
-				<state_interface name="position">
-					<param name="intitial_value">0.0</param>
-				</state_interface>
-				<state_interface name="velocity"/>
-				<state_interface name="effort"/>
-			</joint>
-			<joint name="${prefix}_wheel_joint">
-				<command_interface name="velocity">
-					<param name="min">-20</param>
-					<param name="max">20</param>
-				</command_interface>
-				<state_interface name="position"/>
-				<state_interface name="velocity"/>
-				<state_interface name="effort"/>
-			</joint>
-		</ros2_control>-->
     </xacro:macro>
 </robot>

Commit message: add visualization for test

File: xacro/wheel_macro.xacro (robot description, xacro)
@@ -50,4 +50,16 @@
 			</collision>
 		</link>
+		<joint name="${prefix}_test" type="fixed">
+			<origin xyz="0 0 0.03"/>
+			<parent link="${prefix}_wheel_link"/>
+			<child link="${prefix}_test_link"/>
+		</joint>
+		<link name="${prefix}_test_link">
+			<visual>
+				<geometry>
+					<box size="0.05 0.05 0.03"/>
+				</geometry>
+			</visual>
+		</link>
 		<gazebo reference="${prefix}_wheel_link">
 			<mu1 value="2.5"/>

Commit message: remove test wheel object

File: xacro/wheel_macro.xacro (robot description, xacro)
@@ -50,16 +50,4 @@
 			</collision>
 		</link>
-		<joint name="${prefix}_test" type="fixed">
-			<origin xyz="0 0 0.03"/>
-			<parent link="${prefix}_wheel_link"/>
-			<child link="${prefix}_test_link"/>
-		</joint>
-		<link name="${prefix}_test_link">
-			<visual>
-				<geometry>
-					<box size="0.05 0.05 0.03"/>
-				</geometry>
-			</visual>
-		</link>
 		<gazebo reference="${prefix}_wheel_link">
 			<mu1 value="2.5"/>
