Commit message: back up commit

File: xacro/control_macro.xacro (robot description, xacro)
@@ -86,16 +86,4 @@
 				<state_interface name="effort"/>
 			</joint>
-			<sensor name="imu_sensor">
-				<state_interface name="orientation.x"/>
-				<state_interface name="orientation.y"/>
-				<state_interface name="orientation.z"/>
-				<state_interface name="orientation.w"/>
-				<state_interface name="angular_velocity.x"/>
-				<state_interface name="angular_velocity.y"/>
-				<state_interface name="angular_velocity.z"/>
-				<state_interface name="linear_acceleration.x"/>
-				<state_interface name="linear_acceleration.y"/>
-				<state_interface name="linear_acceleration.z"/>
-			</sensor>
 		</ros2_control>
 	</xacro:macro>

File: xacro/omni_robot.xacro (robot description, xacro)
@@ -32,67 +32,15 @@
 		</collision>
 	</link>
-	<joint name="imu_join" type="fixed">
-		<origin xyz="0 0 0" rpy="0 0 0"/>
-		<parent link="body_link"/>
-		<child link="imu_link"/>
-	</joint>
-	<link name="imu_link"/>
-	<gazebo reference="imu_link">
-		<sensor name="imu_sensor" type="imu">
-			<always_on>1</always_on>
-			<update_rate>10.0</update_rate>
-		</sensor>
-	</gazebo>
-	<joint name="scan_joint" type="fixed">
-		<origin xyz="0 0.2 -0.04" rpy="0 0 0"/>
-		<parent link="body_link"/>
-		<child link="laser_link"/>
-	</joint>
-	<link name="laser_link">
-		<visual>
-			<cylinder radius="0.04" length="0.02"/>
-		</visual>
-	</link>
-	<gazebo reference="laser_link">
-		<sensor name="laser_link" type="ray">
-			<topic>scan</topic>
-			<ignition_frame_id>laser_link</ignition_frame_id>
-			<update_rate>5</update_rate>
-			<ray>
-				<scan>
-					<horizontal>
-						<samples>360</samples>
-						<resolution>1</resolution>
-						<min_angle>0</min_angle>
-						<max_angle>6.28</max_angle>
-					</horizontal>
-				</scan>
-				<range>
-					<min>0.120000</min>
-					<max>20.0</max>
-					<resolution>0.015000</resolution>
-				</range>
-				<frame_id>laser_link</frame_id>
-				<noise>
-					<type>gaussian</type>
-					<mean>0.0</mean>
-					<stddev>0.01</stddev>
-				</noise>
-			</ray>
-			<always_on>true</always_on>
-			<visualize>false</visualize>
-			<plugin name="turtlebot3_laserscan" filename="libgazebo_ros_ray_sensor.so">
-				<ros>
-					<remapping>~/out:=scan</remapping>
-				</ros>
-				<output_type>sensor_msgs/LaserScan</output_type>
-				<frame_name>laser_link</frame_name>
-			</plugin>
-		</sensor>
-	</gazebo>
+	<xacro:imu_macro prefix="imu" parent="body_link" xyz="0 0 0" rpy="0 0 0"/>
+	<xacro:lidar_macro prefix="laser" parent="body_link" xyz="0 0.2 -0.04" rpy="0 0 0"/>
 	<xacro:wheel_macro prefix="fr_wheel" parent="body_link" xyz="0.2 0.2 -0.06"/>
 	<xacro:wheel_macro prefix="fl_wheel" parent="body_link" xyz="-0.2 0.2 -0.06"/>
 	<xacro:wheel_macro prefix="bl_wheel" parent="body_link" xyz="-0.2 -0.2 -0.06"/>
 	<xacro:wheel_macro prefix="br_wheel" parent="body_link" xyz="0.2 -0.2 -0.06"/>
+	<ros2_control name="GazeboSystem" type="system">
+		<hardware>
+			<plugin>gazebo_ros2_control/GazeboSystem</plugin>
+		</hardware>
+	</ros2_control>
 	<xacro:control_macro/>
 	<gazebo>

Commit message: clean up xacro files

File: xacro/control_macro.xacro (robot description, xacro)
@@ -1,90 +1,25 @@
 <?xml version="1.0" encoding="utf-8"?>
 <robot xmlns:xacro="https://www.ros.org/wiki/xacro">
-	<xacro:macro name="control_macro">
-		<ros2_control name="GazeboSystem" type="system">
-			<hardware>
-				<plugin>gazebo_ros2_control/GazeboSystem</plugin>
-			</hardware>
-			<joint name="fr_wheel_rotate_joint">
-				<command_interface name="position">
-					<param name="min">-15</param>
-					<param name="max">15</param>
-				</command_interface>
-				<state_interface name="position">
-					<param name="intitial_value">0.0</param>
-				</state_interface>
-				<state_interface name="velocity"/>
-				<state_interface name="effort"/>
-			</joint>
-			<joint name="fr_wheel_wheel_joint">
-				<command_interface name="velocity">
-					<param name="min">-20</param>
-					<param name="max">20</param>
-				</command_interface>
-				<state_interface name="position"/>
-				<state_interface name="velocity"/>
-				<state_interface name="effort"/>
-			</joint>
-			<joint name="fl_wheel_rotate_joint">
-				<command_interface name="position">
-					<param name="min">-15</param>
-					<param name="max">15</param>
-				</command_interface>
-				<state_interface name="position">
-					<param name="intitial_value">0.0</param>
-				</state_interface>
-				<state_interface name="velocity"/>
-				<state_interface name="effort"/>
-			</joint>
-			<joint name="fl_wheel_wheel_joint">
-				<command_interface name="velocity">
-					<param name="min">-20</param>
-					<param name="max">20</param>
-				</command_interface>
-				<state_interface name="position"/>
-				<state_interface name="velocity"/>
-				<state_interface name="effort"/>
-			</joint>
-			<joint name="bl_wheel_rotate_joint">
-				<command_interface name="position">
-					<param name="min">-15</param>
-					<param name="max">15</param>
-				</command_interface>
-				<state_interface name="position">
-					<param name="intitial_value">0.0</param>
-				</state_interface>
-				<state_interface name="velocity"/>
-				<state_interface name="effort"/>
-			</joint>
-			<joint name="bl_wheel_wheel_joint">
-				<command_interface name="velocity">
-					<param name="min">-20</param>
-					<param name="max">20</param>
-				</command_interface>
-				<state_interface name="position"/>
-				<state_interface name="velocity"/>
-				<state_interface name="effort"/>
-			</joint>
-			<joint name="br_wheel_rotate_joint">
-				<command_interface name="position">
-					<param name="min">-15</param>
-					<param name="max">15</param>
-				</command_interface>
-				<state_interface name="position">
-					<param name="intitial_value">0.0</param>
-				</state_interface>
-				<state_interface name="velocity"/>
-				<state_interface name="effort"/>
-			</joint>
-			<joint name="br_wheel_wheel_joint">
-				<command_interface name="velocity">
-					<param name="min">-20</param>
-					<param name="max">20</param>
-				</command_interface>
-				<state_interface name="position"/>
-				<state_interface name="velocity"/>
-				<state_interface name="effort"/>
-			</joint>
-		</ros2_control>
+	<xacro:macro name="wheel_control_macro" params="prefix">
+		<joint name="${prefix}_rotate_joint">
+			<command_interface name="position">
+				<param name="min">-15</param>
+				<param name="max">15</param>
+			</command_interface>
+			<state_interface name="position">
+				<param name="intitial_value">0.0</param>
+			</state_interface>
+			<state_interface name="velocity"/>
+			<state_interface name="effort"/>
+		</joint>
+		<joint name="${prefix}_wheel_joint">
+			<command_interface name="velocity">
+				<param name="min">-20</param>
+				<param name="max">20</param>
+			</command_interface>
+			<state_interface name="position"/>
+			<state_interface name="velocity"/>
+			<state_interface name="effort"/>
+		</joint>
 	</xacro:macro>
 </robot>

File: xacro/omni_robot.xacro (robot description, xacro)
@@ -4,4 +4,5 @@
 	<xacro:include filename="$(find omni_sim)/xacro/wheel_macro.xacro"/>
 	<xacro:include filename="$(find omni_sim)/xacro/control_macro.xacro"/>
+	<xacro:include filename="$(find omni_sim)/xacro/sensor_macro.xacro"/>
 	<link name="base_footprint"/>
 	<joint name="base_joint" type="fixed">
@@ -42,6 +43,10 @@
 			<plugin>gazebo_ros2_control/GazeboSystem</plugin>
 		</hardware>
+		<xacro:wheel_control_macro prefix="fr_wheel"/>
+		<xacro:wheel_control_macro prefix="fl_wheel"/>
+		<xacro:wheel_control_macro prefix="bl_wheel"/>
+		<xacro:wheel_control_macro prefix="br_wheel"/>
+		<xacro:imu_control_macro prefix="imu"/>
 	</ros2_control>
-	<xacro:control_macro/>
 	<gazebo>
 		<plugin filename="libgazebo_ros2_control.so" name="gazebo_ros2_control">

File: xacro/sensor_macro.xacro (robot description, xacro)
@@ -1,5 +1,5 @@
 <?xml version="1.0" encoding="utf-8"?>
 <robot xmlns:xacro="https://www.ros.org/wiki/xacro">
-	<xacro:macro name="imu_macro" param="parent prefix xyz rpy">
+	<xacro:macro name="imu_macro" params="parent prefix xyz rpy">
 		<joint name="${prefix}_join" type="fixed">
 			<origin xyz="${xyz}" rpy="${rpy}"/>
@@ -14,20 +14,20 @@
 			</sensor>
 		</gazebo>
-		<ros2_control>
-			<sensor name="imu_sensor">
-				<state_interface name="orientation.x"/>
-				<state_interface name="orientation.y"/>
-				<state_interface name="orientation.z"/>
-				<state_interface name="orientation.w"/>
-				<state_interface name="angular_velocity.x"/>
-				<state_interface name="angular_velocity.y"/>
-				<state_interface name="angular_velocity.z"/>
-				<state_interface name="linear_acceleration.x"/>
-				<state_interface name="linear_acceleration.y"/>
-				<state_interface name="linear_acceleration.z"/>
-			</sensor>
-		</ros2_control>
 	</xacro:macro>
-	<xacro:macro name="lidar_macro" param="parent prefix xyz rpy">
+	<xacro:macro name="imu_control_macro" params="prefix">
+		<sensor name="${prefix}_sensor">
+			<state_interface name="orientation.x"/>
+			<state_interface name="orientation.y"/>
+			<state_interface name="orientation.z"/>
+			<state_interface name="orientation.w"/>
+			<state_interface name="angular_velocity.x"/>
+			<state_interface name="angular_velocity.y"/>
+			<state_interface name="angular_velocity.z"/>
+			<state_interface name="linear_acceleration.x"/>
+			<state_interface name="linear_acceleration.y"/>
+			<state_interface name="linear_acceleration.z"/>
+		</sensor>
+	</xacro:macro>
+	<xacro:macro name="lidar_macro" params="parent prefix xyz rpy">
 		<joint name="${prefix}_joint" type="fixed">
 			<origin xyz="0 0.2 -0.04" rpy="0 0 0"/>
