Commit message: fix bug  with the laser link not appiear

File: xacro/sensor_macro.xacro (robot description, xacro)
@@ -37,5 +37,7 @@
 		<link name="${prefix}_link">
 			<visual>
-				<cylinder radius="0.04" length="0.02"/>
+				<geometry>
+					<cylinder radius="0.04" length="0.02"/>
+				</geometry>
 			</visual>
 		</link>
