Commit message: writing xacro adjusting to ros2control

File: xacro/omni_robot.xacro (robot description, xacro)
@@ -2,2 +2,32 @@
 <robot name="omni_robot" xmlns:xacro="https://ros.org/wiki/xacro">
 	<xacro:arg name="robot_name" default="dtw_robot"/>
+	<xacro:include filename="($find omni_sim)/xacro/wheel_macro.xacro" />
+	<link name="base_link"/>
+	<joint name="body_joint" type="fix">
+		<parent link="base_link"/>
+		<child link="body_link"/>
+		<origin xyz="0 0 0.11" rpy="0 0 0"/>
+	</joint>
+	<link name="body_link">
+		<inertial>
+			<origin xyz="0 0 0" rpy="0 0 0"/>
+			<mass value="2.0"/>
+			<inertia ixx="0.001" ixy="0" ixz="0" iyy="0.001" iyz="0" izz="0.002"/>
+		</inertial>
+		<visual>
+			<geometry>
+				<box size="0.5 0.5 0.06"/>
+			</geometry>
+		</visual>
+		<collision>
+			<geometry>
+				<box size="0.5 0.5 0.06"/>
+			</geometry>
+		</collision>
+	</link>
+	<xacro:wheel_macro prefix="fr_wheel" parent="body_link" xyz="0.2 0.2 -0.06"/>
+	<xacro:wheel_macro prefix="fl_wheel" parent="body_link" xyz="0.2 -0.2 -0.06"/>
+	<xacro:wheel_macro prefix="bl_wheel" parent="body_link" xyz="-0.2 -0.2 -0.06"/>
+	<xacro:wheel_macro prefix="br_wheel" parent="body_link" xyz="-0.2 0.2 -0.06"/>
+	<gazebo>
+		<plugin filename="libgazebo_ros2_control.so" name="gazebo_ros2_control">

File: xacro/wheel_macro.xacro (robot description, xacro)
@@ -36,5 +36,5 @@
 		</link>
 		<joint name="${prefix}_wheel_joint" type="continuous">
-			<origin xyz="0 0 -0.3" rpy="${radians{-90}} 0 0" />
+			<origin xyz="0 0 -0.03" rpy="${radians{-90}} 0 0" />
 			<parent link="${prefix}_rotate_link" />
 			<child link="${prefix}_wheel_link" />
@@ -42,12 +42,17 @@
 			<axis xyz="0 0 1" />
 		</joint>
-		<transmission name="{prefix}_wheel_trans">
-			<type>transmitssion_interface/SimpleTransmission</type>
+		<ros2_control name="GazeboSystem" type="system">
+			<hardware>
+				<plugin>gazebo_ros2_control/GazeboSystem</plugin>
+			</hardware>
 			<joint name="{prefix}_wheel_joint">
-				<hardwareInterface>hardware_interface/VelocityJointInterface</hardwareInterface>
+				<command_interface name="velocity">
+					<param name="min">-20</param>
+					<param name="max">20<param>
+				</command_interface>
+				<state_interface name="position"/>
+				<state_interface name="velocity"/>
+				<state_interface name="effort"/>
 			</joint>
-			<actuator name="${prefix}_wheel_motor">
-				<hardwareInterface>hardware_interface/VelocityJointInterface</hardareInterface>
-			</actuator>
 		</transmission>
 		<link name="{prefix}_wheel_link">

Commit message: temporary complete writing xacro. remain debuging

File: xacro/omni_robot.xacro (robot description, xacro)
@@ -32,2 +32,6 @@
 	<gazebo>
 		<plugin filename="libgazebo_ros2_control.so" name="gazebo_ros2_control">
+			<parameters>$(find omni_sim)/config/omni_sim.yaml</parameters>
+		</plugin>
+	</gazebo>
+</robot>

File: xacro/wheel_macro.xacro (robot description, xacro)
@@ -42,18 +42,4 @@
 			<axis xyz="0 0 1" />
 		</joint>
-		<ros2_control name="GazeboSystem" type="system">
-			<hardware>
-				<plugin>gazebo_ros2_control/GazeboSystem</plugin>
-			</hardware>
-			<joint name="{prefix}_wheel_joint">
-				<command_interface name="velocity">
-					<param name="min">-20</param>
-					<param name="max">20<param>
-				</command_interface>
-				<state_interface name="position"/>
-				<state_interface name="velocity"/>
-				<state_interface name="effort"/>
-			</joint>
-		</transmission>
 		<link name="{prefix}_wheel_link">
 			<inertial>
@@ -79,4 +65,29 @@
 			<kd value="10"/>
 		</gazebo>
+		<ros2_control name="GazeboSystem" type="system">
+			<hardware>
+				<plugin>gazebo_ros2_control/GazeboSystem</plugin>
+			</hardware>
+			<joint name="{prefix}_rotate_joint">
+				<command_interface name="position">
+					<param name="min">-15</param>
+					<param name="max">15</param>
+				</command_interface>
+				<state_interface name="position">
+					<param name="intitial_value">0.0</param>
+				</state_interface>
+				<state_interface name="velocity"/>
+				<state_interface name="effort"/>
+			</joint>
+			<joint name="{prefix}_wheel_joint">
+				<command_interface name="velocity">
+					<param name="min">-20</param>
+					<param name="max">20<param>
+				</command_interface>
+				<state_interface name="position"/>
+				<state_interface name="velocity"/>
+				<state_interface name="effort"/>
+			</joint>
+		</ros2_control>
     </xacro:macro>
 </robot>

Commit message: spawn robot in gazebo suceeded

File: xacro/omni_robot.xacro (robot description, xacro)
@@ -1,8 +1,8 @@
 <?xml version="1.0"?>
 <robot name="omni_robot" xmlns:xacro="https://ros.org/wiki/xacro">
-	<xacro:arg name="robot_name" default="dtw_robot"/>
-	<xacro:include filename="($find omni_sim)/xacro/wheel_macro.xacro" />
+	<xacro:arg name="robot_name" default="omni_robot"/>
+	<xacro:include filename="$(find omni_sim)/xacro/wheel_macro.xacro" />
 	<link name="base_link"/>
-	<joint name="body_joint" type="fix">
+	<joint name="body_joint" type="fixed">
 		<parent link="base_link"/>
 		<child link="body_link"/>

File: xacro/wheel_macro.xacro (robot description, xacro)
@@ -2,5 +2,5 @@
 <robot name="omni_robot" xmlns:xacro="https://ros.org/wiki/xacro">
     <xacro:macro name="wheel_macro" params="parent prefix xyz">
-		<joint="${prefix}_rotate_joint" type="continuous">
+		<joint name="${prefix}_rotate_joint" type="continuous">
 			<origin xyz="${xyz}" rpy="0 0 0" />
 			<parent link="${parent}" />
@@ -9,14 +9,5 @@
 			<axis xyz="0 0 1" />
 		</joint>
-		<transmission name="${prefix}_rotate_trans">
-			<type>transmitssion_interface/SimpleTransmission</type>
-			<joint name="${prefix}_rotate_joint">
-				<hardwareInterface>hardware_interface/PositinJointInterface</hardwareInterface>
-			</joint>
-			<actuator name="{prefix}_rotate_motor">
-				<hardwareInterface>hardware_interface/PositinJointInterface</hardwareInterface>
-			</actuator>
-		</transmission>
-		<link name="{prefix}_rotate_link">
+		<link name="${prefix}_rotate_link">
 			<inertial>
 				<origin xyz="0 0 0" rpy="0 0 0"/>
@@ -26,21 +17,21 @@
 			<visual>
 				<geometry>
-					<cylinder radius="0.10" length="0.03" />
+					<cylinder radius="0.05" length="0.03" />
 				</geometry>
 			</visual>
 			<collision>
 				<geometry>
-					<cylinder radius="0.10" length="0.03" />
+					<cylinder radius="0.05" length="0.03" />
 				</geometry>
 			</collision>
 		</link>
 		<joint name="${prefix}_wheel_joint" type="continuous">
-			<origin xyz="0 0 -0.03" rpy="${radians{-90}} 0 0" />
+			<origin xyz="0 0 -0.03" rpy="${radians(-90)} 0 0" />
 			<parent link="${prefix}_rotate_link" />
 			<child link="${prefix}_wheel_link" />
-			<limit velocity="50" effor="2.0" />
+			<limit velocity="50" effort="2.0" />
 			<axis xyz="0 0 1" />
 		</joint>
-		<link name="{prefix}_wheel_link">
+		<link name="${prefix}_wheel_link">
 			<inertial>
 				<origin xyz="0 0 0" rpy="0 0 0" />
@@ -50,10 +41,10 @@
 			<visual>
 				<geometry>
-					<cylinder radius="0.10" length="0.03" />
+					<cylinder radius="0.05" length="0.03" />
 				</geometry>
 			</visual>
 			<collision>
 				<geometry>
-					<cylinder radius="0.10" length="0.03" />
+					<cylinder radius="0.05" length="0.03" />
 				</geometry>
 			</collision>
@@ -83,5 +74,5 @@
 				<command_interface name="velocity">
 					<param name="min">-20</param>
-					<param name="max">20<param>
+					<param name="max">20</param>
 				</command_interface>
 				<state_interface name="position"/>

Commit message: backup commit

File: xacro/omni_robot.xacro (robot description, xacro)
@@ -30,4 +30,89 @@
 	<xacro:wheel_macro prefix="bl_wheel" parent="body_link" xyz="-0.2 -0.2 -0.06"/>
 	<xacro:wheel_macro prefix="br_wheel" parent="body_link" xyz="-0.2 0.2 -0.06"/>
+	<ros2_control name="GazeboSystem" type="system">
+		<hardware>
+			<plugin>gazebo_ros2_control/GazeboSystem</plugin>
+		</hardware>
+		<joint name="fr_wheel_rotate_joint">
+			<command_interface name="position">
+				<param name="min">-15</param>
+				<param name="max">15</param>
+			</command_interface>
+			<state_interface name="position">
+				<param name="intitial_value">0.0</param>
+			</state_interface>
+			<state_interface name="velocity"/>
+			<state_interface name="effort"/>
+		</joint>
+		<joint name="fr_wheel_wheel_joint">
+			<command_interface name="velocity">
+				<param name="min">-20</param>
+				<param name="max">20</param>
+			</command_interface>
+			<state_interface name="position"/>
+			<state_interface name="velocity"/>
+			<state_interface name="effort"/>
+		</joint>
+		<joint name="fl_wheel_rotate_joint">
+			<command_interface name="position">
+				<param name="min">-15</param>
+				<param name="max">15</param>
+			</command_interface>
+			<state_interface name="position">
+				<param name="intitial_value">0.0</param>
+			</state_interface>
+			<state_interface name="velocity"/>
+			<state_interface name="effort"/>
+		</joint>
+		<joint name="fl_wheel_wheel_joint">
+			<command_interface name="velocity">
+				<param name="min">-20</param>
+				<param name="max">20</param>
+			</command_interface>
+			<state_interface name="position"/>
+			<state_interface name="velocity"/>
+			<state_interface name="effort"/>
+		</joint>
+		<joint name="bl_wheel_rotate_joint">
+			<command_interface name="position">
+				<param name="min">-15</param>
+				<param name="max">15</param>
+			</command_interface>
+			<state_interface name="position">
+				<param name="intitial_value">0.0</param>
+			</state_interface>
+			<state_interface name="velocity"/>
+			<state_interface name="effort"/>
+		</joint>
+		<joint name="bl_wheel_wheel_joint">
+			<command_interface name="velocity">
+				<param name="min">-20</param>
+				<param name="max">20</param>
+			</command_interface>
+			<state_interface name="position"/>
+			<state_interface name="velocity"/>
+			<state_interface name="effort"/>
+		</joint>
+		<joint name="br_wheel_rotate_joint">
+			<command_interface name="position">
+				<param name="min">-15</param>
+				<param name="max">15</param>
+			</command_interface>
+			<state_interface name="position">
+				<param name="intitial_value">0.0</param>
+			</state_interface>
+			<state_interface name="velocity"/>
+			<state_interface name="effort"/>
+		</joint>
+		<joint name="br_wheel_wheel_joint">
+			<command_interface name="velocity">
+				<param name="min">-20</param>
+				<param name="max">20</param>
+			</command_interface>
+			<state_interface name="position"/>
+			<state_interface name="velocity"/>
+			<state_interface name="effort"/>
+		</joint>
+	</ros2_control>
 	<gazebo>
 		<plugin filename="libgazebo_ros2_control.so" name="gazebo_ros2_control">

File: xacro/wheel_macro.xacro (robot description, xacro)
@@ -56,5 +56,5 @@
 			<kd value="10"/>
 		</gazebo>
-		<ros2_control name="GazeboSystem" type="system">
+		<!--<ros2_control name="GazeboSystem" type="system">
 			<hardware>
 				<plugin>gazebo_ros2_control/GazeboSystem</plugin>
@@ -80,5 +80,5 @@
 				<state_interface name="effort"/>
 			</joint>
-		</ros2_control>
+		</ros2_control>-->
     </xacro:macro>
 </robot>

Commit message: add imu

File: xacro/omni_robot.xacro (robot description, xacro)
@@ -26,4 +26,16 @@
 		</collision>
 	</link>
+	<joint name="imu_join" type="fixed">
+		<origin xyz="0 0 0" rpy="0 0 0"/>
+		<parent link="body_link"/>
+		<child link="imu_link"/>
+	</joint>
+	<link name="imu_link"/>
+	<gazebo reference="imu_link">
+		<sensor name="imu_sensor" type="imu">
+			<always_on>1</always_on>
+			<update_rate>10.0</update_rate>
+		</sensor>
+	</gazebo>
 	<xacro:wheel_macro prefix="fr_wheel" parent="body_link" xyz="0.2 0.2 -0.06"/>
 	<xacro:wheel_macro prefix="fl_wheel" parent="body_link" xyz="0.2 -0.2 -0.06"/>
@@ -114,4 +126,16 @@
 			<state_interface name="effort"/>
 		</joint>
+		<sensor name="imu_sensor">
+			<state_interface name="orientation.x"/>
+			<state_interface name="orientation.y"/>
+			<state_interface name="orientation.z"/>
+			<state_interface name="orientation.w"/>
+			<state_interface name="angular_velocity.x"/>
+			<state_interface name="angular_velocity.y"/>
+			<state_interface name="angular_velocity.z"/>
+			<state_interface name="linear_acceleration.x"/>
+			<state_interface name="linear_acceleration.y"/>
+			<state_interface name="linear_acceleration.z"/>
+		</sensor>
 	</ros2_control>
 	<gazebo>

Commit message: split control xacro file

File: xacro/omni_robot.xacro (robot description, xacro)
@@ -2,5 +2,6 @@
 <robot name="omni_robot" xmlns:xacro="https://ros.org/wiki/xacro">
 	<xacro:arg name="robot_name" default="omni_robot"/>
-	<xacro:include filename="$(find omni_sim)/xacro/wheel_macro.xacro" />
+	<xacro:include filename="$(find omni_sim)/xacro/wheel_macro.xacro"/>
+	<xacro:include filename="$(find omni_sim)/xacro/control_macro.xacro"/>
 	<link name="base_link"/>
 	<joint name="body_joint" type="fixed">
@@ -42,101 +43,5 @@
 	<xacro:wheel_macro prefix="bl_wheel" parent="body_link" xyz="-0.2 -0.2 -0.06"/>
 	<xacro:wheel_macro prefix="br_wheel" parent="body_link" xyz="-0.2 0.2 -0.06"/>
-	<ros2_control name="GazeboSystem" type="system">
-		<hardware>
-			<plugin>gazebo_ros2_control/GazeboSystem</plugin>
-		</hardware>
-		<joint name="fr_wheel_rotate_joint">
-			<command_interface name="position">
-				<param name="min">-15</param>
-				<param name="max">15</param>
-			</command_interface>
-			<state_interface name="position">
-				<param name="intitial_value">0.0</param>
-			</state_interface>
-			<state_interface name="velocity"/>
-			<state_interface name="effort"/>
-		</joint>
-		<joint name="fr_wheel_wheel_joint">
-			<command_interface name="velocity">
-				<param name="min">-20</param>
-				<param name="max">20</param>
-			</command_interface>
-			<state_interface name="position"/>
-			<state_interface name="velocity"/>
-			<state_interface name="effort"/>
-		</joint>
-		<joint name="fl_wheel_rotate_joint">
-			<command_interface name="position">
-				<param name="min">-15</param>
-				<param name="max">15</param>
-			</command_interface>
-			<state_interface name="position">
-				<param name="intitial_value">0.0</param>
-			</state_interface>
-			<state_interface name="velocity"/>
-			<state_interface name="effort"/>
-		</joint>
-		<joint name="fl_wheel_wheel_joint">
-			<command_interface name="velocity">
-				<param name="min">-20</param>
-				<param name="max">20</param>
-			</command_interface>
-			<state_interface name="position"/>
-			<state_interface name="velocity"/>
-			<state_interface name="effort"/>
-		</joint>
-		<joint name="bl_wheel_rotate_joint">
-			<command_interface name="position">
-				<param name="min">-15</param>
-				<param name="max">15</param>
-			</command_interface>
-			<state_interface name="position">
-				<param name="intitial_value">0.0</param>
-			</state_interface>
-			<state_interface name="velocity"/>
-			<state_interface name="effort"/>
-		</joint>
-		<joint name="bl_wheel_wheel_joint">
-			<command_interface name="velocity">
-				<param name="min">-20</param>
-				<param name="max">20</param>
-			</command_interface>
-			<state_interface name="position"/>
-			<state_interface name="velocity"/>
-			<state_interface name="effort"/>
-		</joint>
-		<joint name="br_wheel_rotate_joint">
-			<command_interface name="position">
-				<param name="min">-15</param>
-				<param name="max">15</param>
-			</command_interface>
-			<state_interface name="position">
-				<param name="intitial_value">0.0</param>
-			</state_interface>
-			<state_interface name="velocity"/>
-			<state_interface name="effort"/>
-		</joint>
-		<joint name="br_wheel_wheel_joint">
-			<command_interface name="velocity">
-				<param name="min">-20</param>
-				<param name="max">20</param>
-			</command_interface>
-			<state_interface name="position"/>
-			<state_interface name="velocity"/>
-			<state_interface name="effort"/>
-		</joint>
-		<sensor name="imu_sensor">
-			<state_interface name="orientation.x"/>
-			<state_interface name="orientation.y"/>
-			<state_interface name="orientation.z"/>
-			<state_interface name="orientation.w"/>
-			<state_interface name="angular_velocity.x"/>
-			<state_interface name="angular_velocity.y"/>
-			<state_interface name="angular_velocity.z"/>
-			<state_interface name="linear_acceleration.x"/>
-			<state_interface name="linear_acceleration.y"/>
-			<state_interface name="linear_acceleration.z"/>
-		</sensor>
-	</ros2_control>
+	<xacro:control_macro/>
 	<gazebo>
 		<plugin filename="libgazebo_ros2_control.so" name="gazebo_ros2_control">

Commit message: add base_footprint for navigation

File: xacro/omni_robot.xacro (robot description, xacro)
@@ -4,9 +4,14 @@
 	<xacro:include filename="$(find omni_sim)/xacro/wheel_macro.xacro"/>
 	<xacro:include filename="$(find omni_sim)/xacro/control_macro.xacro"/>
+	<link name="base_footprint"/>
+	<joint name="base_joint" type="fixed">
+		<parent link="base_footprint"/>
+		<child link="base_link"/>
+	</joint>
 	<link name="base_link"/>
 	<joint name="body_joint" type="fixed">
 		<parent link="base_link"/>
 		<child link="body_link"/>
-		<origin xyz="0 0 0.11" rpy="0 0 0"/>
+		<origin xyz="0 0 0.15" rpy="0 0 0"/>
 	</joint>
 	<link name="body_link">
@@ -39,4 +44,46 @@
 		</sensor>
 	</gazebo>
+	<joint name="scan_joint" type="fixed">
+		<origin xyz="0 0.2 -0.04" rpy="0 0 0"/>
+		<parent link="body_link"/>
+		<child link="laser_link"/>
+	</joint>
+	<link name="laser_link">
+		<visual>
+			<cylinder radius="0.04" length="0.02"/>
+		</visual>
+	</link>
+	<gazebo reference="laser_link">
+		<sensor name="laser_link" type="ray">
+			<topic>scan</topic>
+			<ignition_frame_id>laser_link</ignition_frame_id>
+			<update_rate>5</update_rate>
+			<ray>
+				<scan>
+					<horizontal>
+						<samples>360</samples>
+						<resolution>1</resolution>
+						<min_angle>0</min_angle>
+						<max_angle>6.28</max_angle>
+					</horizontal>
+				</scan>
+				<range>
+					<min>0.120000</min>
+					<max>20.0</max>
+					<resolution>0.015000</resolution>
+				</range>
+				<frame_id>/laser_link</frame_id>
+			</ray>
+			<always_on>true</always_on>
+			<visualize>false</visualize>
+			<plugin name="turtlebot3_laserscan" filename="libgazebo_ros_ray_sensor.so">
+				<ros>
+					<remapping>~/out:=scan</remapping>
+				</ros>
+				<output_type>sensor_msgs/LaserScan</output_type>
+				<frame_name>laser_link</frame_name>
+			</plugin>
+		</sensor>
+	</gazebo>
 	<xacro:wheel_macro prefix="fr_wheel" parent="body_link" xyz="0.2 0.2 -0.06"/>
 	<xacro:wheel_macro prefix="fl_wheel" parent="body_link" xyz="0.2 -0.2 -0.06"/>

Commit message: adjust sensor position

File: xacro/omni_robot.xacro (robot description, xacro)
@@ -34,5 +34,5 @@
 	</link>
 	<xacro:imu_macro prefix="imu" parent="body_link" xyz="0 0 0" rpy="0 0 0"/>
-	<xacro:lidar_macro prefix="laser" parent="body_link" xyz="0 0.2 -0.04" rpy="0 0 0"/>
+	<xacro:lidar_macro prefix="laser" parent="body_link" xyz="0 0.2 -0.10" rpy="0 0 0"/>
 	<xacro:wheel_macro prefix="fr_wheel" parent="body_link" xyz="0.2 0.2 -0.06"/>
 	<xacro:wheel_macro prefix="fl_wheel" parent="body_link" xyz="-0.2 0.2 -0.06"/>

File: xacro/sensor_macro.xacro (robot description, xacro)
@@ -31,5 +31,5 @@
 	<xacro:macro name="lidar_macro" params="parent prefix xyz rpy">
 		<joint name="${prefix}_joint" type="fixed">
-			<origin xyz="0 0.2 -0.04" rpy="0 0 0"/>
+			<origin xyz="${xyz}" rpy="${rpy}"/>
 			<parent link="${parent}"/>
 			<child link="${prefix}_link"/>
